File: _autosave-backplane.kicad_pcb (KiCad board)
At the start: 4 copper layers, 110 x 90 mm, 57 parts, among them IC1 SiC437AED-T1-GE3, J1 46010-0622, J2 46010-0622, J4 212520-1006, J5 XT60PW-F

Commit message: more drcs out
last error is naming convention - after will neaten everything up + add a switch then should be done
Parts:
- moved R24 0.95 mm to (124.0, 124.0)
- moved R26 0.95 mm to (124.0, 124.9)
- moved C51 0.78 mm to (114.0, 127.2)
Routing:
- net RBUS_uC_V: track 5.63 -> 31.3 mm, vias 1 -> 2
- net /buckC/Vdd: track 6.36 -> 14.9 mm
- net Net-(IC1-EN): track 1.59 -> 9.01 mm, vias 0 -> 2
- net /buckC/SW: track 0.00 -> 7.23 mm
- net /buckC/MODE_1: track 2.17 -> 3.12 mm
- net /buckC/MODE_2: track 1.96 -> 2.91 mm
- net Net-(C51-Pad2): track 1.72 -> 2.50 mm
- added copper zone on F.Cu, net +3.3V
- added copper zone on F.Cu, net /buckC/SW

Commit message: filleted
to add switches then next review
Parts:
- moved J2 0.22 mm to (151.2, 80.8)
- moved J1 0.14 mm to (151.1, 104.0)
Connections:
- C47 pad 1: Net-(IC1-EN) -> +12V
- C49 pad 1: Net-(IC1-EN) -> +12V
- IC1 pad 1: Net-(IC1-EN) -> +12V
- IC1 pad 19: Net-(IC1-EN) -> +12V
- IC1 pad 2: Net-(IC1-EN) -> +12V
- IC1 pad 22: Net-(IC1-EN) -> +12V
- IC1 pad 26: Net-(IC1-EN) -> +12V
Routing:
- net Net-(IC1-EN): track 9.01 -> 0.00 mm, vias 2 -> 0
- net +12V: track 117.3 -> 125.6 mm, vias 10 -> 12
- net CAN_H: track 80.6 -> 78.2 mm
- net +3.3V: track 79.6 -> 80.3 mm
- net GND: track 3.26 -> 2.76 mm
