File: backplane.kicad_pcb (KiCad board)
At the start: 4 copper layers, 110 x 90 mm, 57 parts, among them IC1 SiC437AED-T1-GE3, J1 46010-0622, J2 46010-0622, J4 212520-1006, J5 XT60PW-F

Commit message: filleted
to add switches then next review
Parts:
- moved R24 0.95 mm to (124.0, 124.0)
- moved R26 0.95 mm to (124.0, 124.9)
Routing:
- net RBUS_uC_V: track 3.34 -> 31.3 mm, vias 0 -> 2
- net /buckC/Vdd: track 6.36 -> 14.9 mm
- net Net-(IC1-EN): track 14.3 -> 9.01 mm, vias 0 -> 2
- net /buckC/MODE_1: track 2.17 -> 3.12 mm
- net /buckC/MODE_2: track 1.96 -> 2.91 mm
Changed lines of the file:
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@@
 	(footprint "Resistor_SMD:R_0402_1005Metric"
 		(layer "F.Cu")
-		(at 123.058944 124.944304)
+		(at 124.010982 124.944304)
 		(descr "Resistor SMD 0402 (1005 Metric), square (rectangular) end terminal, IPC_7351 nominal, (Body size source: IPC-SM-782 page 72, https://www.pcb-3d.com/wordpress/wp-content/uploads/ipc-sm-782a_amendment_1_and_2.pdf), generated with kicad-footprint-generator")
 		(tags "resistor")
@@
 	(footprint "Resistor_SMD:R_0402_1005Metric"
 		(layer "F.Cu")
-		(at 123.057962 124 180)
+		(at 124.01 124 180)
 		(descr "Resistor SMD 0402 (1005 Metric), square (rectangular) end terminal, IPC_7351 nominal, (Body size source: IPC-SM-782 page 72, https://www.pcb-3d.com/wordpress/wp-content/uploads/ipc-sm-782a_amendment_1_and_2.pdf), generated with kicad-footprint-generator")
 		(tags "resistor")
@@
 	)
 	(segment
-		(start 120.144962 124.146561)
-		(end 119.544962 123.546561)
-		(width 0.25)
-		(layer "F.Cu")
-		(net 3)
-	)
-	(segment
 		(start 120.731962 124.146561)
-		(end 120.144962 124.146561)
+		(end 122.290361 124.146561)
 		(width 0.25)
 		(layer "F.Cu")
@@
 	)
 	(segment
-		(start 124.325 125.091816)
-		(end 124.325 121.725)
+		(start 120.144962 124.146561)
+		(end 119.544962 123.546561)
 		(width 0.25)
 		(layer "F.Cu")
@@
 	)
 	(segment
-		(start 120.731962 125.746561)
-		(end 123.670255 125.746561)
+		(start 120.731962 124.146561)
+		(end 120.144962 124.146561)
 		(width 0.25)
 		(layer "F.Cu")
@@
 	)
 	(segment
-		(start 121.1 118.5)
-		(end 120.525 118.5)
+		(start 123.5 126)
+		(end 123.246561 125.746561)
 		(width 0.25)
 		(layer "F.Cu")
@@
 	)
 	(segment
-		(start 124.325 121.725)
-		(end 121.1 118.5)
+		(start 122.290361 124.146561)
+		(end 122.436922 124)
 		(width 0.25)
 		(layer "F.Cu")
@@
 	)
 	(segment
-		(start 123.670255 125.746561)
-		(end 124.325 125.091816)
+		(start 123.246561 125.746561)
+		(end 120.731962 125.746561)
 		(width 0.25)
 		(layer "F.Cu")
@@
 		(net 3)
 	)
+	(via
+		(at 123.5 126)
+		(size 0.45)
+		(drill 0.3)
+		(layers "F.Cu" "B.Cu")
+		(free yes)
+		(net 3)
+	)
+	(via
+		(at 122.436922 124)
+		(size 0.45)
+		(drill 0.3)
+		(layers "F.Cu" "B.Cu")
+		(free yes)
+		(net 3)
+	)
+	(segment
+		(start 122.436922 124.936922)
+		(end 123.5 126)
+		(width 0.25)
+		(layer "B.Cu")
+		(net 3)
+	)
+	(segment
+		(start 122.436922 124)
+		(end 122.436922 124.936922)
+		(width 0.25)
+		(layer "B.Cu")
+		(net 3)
+	)
 	(segment
 		(start 151.4 75.5)
@@
 	)
 	(segment
+		(start 124.5 129.5)
+		(end 120.54 129.5)
+		(width 0.25)
+		(layer "F.Cu")
+		(net 9)
+	)
+	(segment
+		(start 120.54 129.5)
+		(end 120.5 129.46)
+		(width 0.25)
+		(layer "F.Cu")
+		(net 9)
+	)
+	(segment
 		(start 119.169962 129.459173)
 		(end 119.170789 129.46)
@@
 	)
 	(segment
-		(start 123.567962 124.943322)
-		(end 123.568944 124.944304)
+		(start 124.52 124.943322)
+		(end 124.520982 124.944304)
 		(width 0.25)
 		(layer "F.Cu")
@@
 	)
 	(segment
+		(start 124.520982 129.479018)
+		(end 124.5 129.5)
+		(width 0.25)
+		(layer "F.Cu")
+		(net 9)
+	)
+	(segment
+		(start 124.520982 124.944304)
+		(end 124.520982 129.479018)
+		(width 0.25)
+		(layer "F.Cu")
+		(net 9)
+	)
+	(segment
 		(start 117.955511 129.46)
 		(end 117.908568 129.506943)
@@
 	)
 	(segment
-		(start 123.567962 124)
-		(end 123.567962 124.943322)
+		(start 124.52 124)
+		(end 124.52 124.943322)
 		(width 0.25)
 		(layer "F.Cu")
@@
 	)
 	(segment
-		(start 121.701401 124.846561)
-		(end 122.547962 124)
+		(start 122.653439 124.846561)
+		(end 123.5 124)
 		(width 0.25)
 		(layer "F.Cu")
@@
 	(segment
 		(start 120.731962 124.846561)
-		(end 121.701401 124.846561)
+		(end 122.653439 124.846561)
 		(width 0.25)
 		(layer "F.Cu")
@@
 	)
 	(segment
-		(start 123.517312 127.5)
+		(start 123.963534 127.053778)
 		(end 123.5 127.517312)
 		(width 0.25)
@@
 	)
 	(segment
+		(start 123.963534 126.603319)
+		(end 123.963534 127.053778)
+		(width 0.25)
+		(layer "F.Cu")
+		(net 22)
+	)
+	(segment
+		(start 107 116.5)
+		(end 106.205848 117.294152)
+		(width 0.25)
+		(layer "F.Cu")
+		(net 22)
+	)
+	(segment
 		(start 122.179249 126.196561)
 		(end 123.5 127.517312)
@@
 	)
 	(segment
-		(start 122.196687 125.296561)
+		(start 106.205848 117.294152)
+		(end 104.5 117.294152)
+		(width 0.25)
+		(layer "F.Cu")
+		(net 22)
+	)
+	(via
+		(at 123.963534 126.603319)
+		(size 0.45)
+		(drill 0.3)
+		(layers "F.Cu" "B.Cu")
+		(free yes)
+		(net 22)
+	)
+	(via
+		(at 107 116.5)
+		(size 0.8)
+		(drill 0.4)
+		(layers "F.Cu" "B.Cu")
+		(net 22)
+	)
+	(segment
+		(start 121.5 120.5)
+		(end 115.5 120.5)
+		(width 0.25)
+		(layer "B.Cu")
+		(net 22)
+	)
+	(segment
+		(start 124.5 123)
+		(end 124 122.5)
+		(width 0.25)
+		(layer "B.Cu")
+		(net 22)
+	)
+	(segment
+		(start 124.5 126)
+		(end 124.5 123)
+		(width 0.25)
+		(layer "B.Cu")
+		(net 22)
+	)
+	(segment
+		(start 115 120)
+		(end 112.5 117.5)
+		(width 0.25)
+		(layer "B.Cu")
+		(net 22)
+	)
+	(segment
+		(start 112.5 117.5)
+		(end 111.5 116.5)
+		(width 0.25)
+		(layer "B.Cu")
+		(net 22)
+	)
+	(segment
+		(start 123.963534 126.603319)
+		(end 124.5 126.066853)
+		(width 0.25)
+		(layer "B.Cu")
+		(net 22)
+	)
+	(segment
+		(start 115.5 120.5)
+		(end 115 120)
+		(width 0.25)
+		(layer "B.Cu")
+		(net 22)
+	)
+	(segment
+		(start 124.5 126.066853)
+		(end 124.5 126)
+		(width 0.25)
+		(layer "B.Cu")
+		(net 22)
+	)
+	(segment
+		(start 124 122.5)
+		(end 122 120.5)
+		(width 0.25)
+		(layer "B.Cu")
+		(net 22)
+	)
+	(segment
+		(start 122 120.5)
+		(end 121.5 120.5)
+		(width 0.25)
+		(layer "B.Cu")
+		(net 22)
+	)
+	(segment
+		(start 111.5 116.5)
+		(end 107 116.5)
+		(width 0.25)
+		(layer "B.Cu")
+		(net 22)
+	)
+	(segment
+		(start 123.148725 125.296561)
 		(end 120.731962 125.296561)
 		(width 0.25)
@@
 	)
 	(segment
-		(start 122.548944 124.944304)
-		(end 122.196687 125.296561)
+		(start 123.500982 124.944304)
+		(end 123.148725 125.296561)
 		(width 0.25)
 		(layer "F.Cu")

Commit message: review overview
half of them sent
Parts:
- moved TP4 20.0 mm to (177.0, 100.6)
- moved TP3 19.2 mm to (117.2, 100.6)
- moved C39 16.5 mm to (134.6, 117.8), turned to -90 degrees
- moved TP2 16.2 mm to (177.0, 95.6)
- moved TP1 15.9 mm to (117.2, 95.4)
- moved C5 7.85 mm to (136.2, 117.8), turned to -90 degrees
- moved C6 7.30 mm to (156.6, 117.6), turned to 90 degrees
- moved C3 4.53 mm to (158.0, 89.0), turned to -90 degrees
- moved J5 4.10 mm to (94.4, 110.8)
- moved C4 3.63 mm to (156.0, 89.0), turned to -90 degrees
- moved C2 3.58 mm to (136.8, 89.2), turned to 90 degrees
- moved 3.3VLED2 1.49 mm to (132.5, 117.0)
- moved R2 1.49 mm to (129.5, 117.0)
- moved J1 0.22 mm to (151.4, 103.9)
- moved J2 0.22 mm to (151.2, 80.8)
Connections:
- C47 pad 1: Net-(IC1-EN) -> +12V
- C49 pad 1: Net-(IC1-EN) -> +12V
- IC1 pad 1: Net-(IC1-EN) -> +12V
- IC1 pad 19: Net-(IC1-EN) -> +12V
- IC1 pad 2: Net-(IC1-EN) -> +12V
- IC1 pad 22: Net-(IC1-EN) -> +12V
- IC1 pad 26: Net-(IC1-EN) -> +12V
Routing:
- net +3.3V: track 79.6 -> 59.5 mm, vias 0 -> 2
- net +12V: track 117.3 -> 103.5 mm, vias 10 -> 13
- net Net-(IC1-EN): track 9.01 -> 0.00 mm, vias 2 -> 0
- net CAN_L: track 79.8 -> 84.7 mm
- net /buckC/Vdd: track 14.9 -> 15.7 mm
- net GND: track 3.26 -> 2.76 mm
- added copper zone on In2.Cu, net +3.3V
- removed copper zone on F.Cu, net +3.3V

Commit message: changes
soham
Parts:
- moved C49 3.85 mm to (121.6, 120.4)
- moved C47 0.10 mm to (122.0, 118.4)

Commit message: made changes
moved some things
Parts:
- moved C49 22.8 mm to (101.5, 109.6), turned to -90 degrees
- moved C47 20.4 mm to (103.6, 109.5), turned to -90 degrees
- moved C41 8.63 mm to (99.0, 115.4), turned to -90 degrees
- moved C40 7.40 mm to (100.5, 115.4), turned to -90 degrees
- moved C29 6.69 mm to (102.1, 115.4), turned to -90 degrees
- moved C45 6.66 mm to (103.6, 115.4), turned to -90 degrees
- moved C43 6.24 mm to (106.6, 115.4)
- moved C42 6.24 mm to (108.1, 115.4)
- moved C44 6.24 mm to (105.1, 115.4)
- moved R5 5.23 mm to (109.5, 115.4)
- moved R6 5.23 mm to (109.5, 113.1)
- moved J1 1.30 mm to (151.4, 105.2)
- moved R27 0.98 mm to (114.0, 131.0), turned to -90 degrees
- moved J2 0.36 mm to (151.2, 80.4)
Routing:
- net +12V: track 103.5 -> 105.7 mm
- net GND: vias 82 -> 84

Commit message: silkscreen
Parts:
- added G***: LOGO, iclr:golden, B.Cu at (139.4, 102.0)
Other:
- outline, holes or cut-outs redrawn
- board text added: "Payload Backplane v1.0"
- board text removed: "Payload Backplane v0.01"
